File: pcb/sat_battery_shield/kicad/_saved_BSAT - Battery Shield.sch (KiCad schematic (older format))
At the start: 65 parts, among them P2 SAT POWER, P3 POWER SAMPLES, Q1 NDS8435A, SW2 SAT ON/OFF, U1 LM78L09, U2 LM78L09, U3 LM78L09, U4 LM78L09, U5 LM78L09, U6 LM78L09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

Commit message: refactor(battery-shield): Rediseño de la placa empleando el regulador de carga MAX1873.
Parts:
- BT1, BT2: symbol Battery -> Battery-RESCUE-BSAT_-_Battery_Shield
Connections:
- net at C23.1, C26.1, Q1.1 (S)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: now also R4.1
Changed lines of the file:
@@
 EESchema Schematic File Version 2
+LIBS:BSAT - Battery Shield-rescue
 LIBS:boscoverysat
 LIBS:power
@@
 $EndDescr
 $Comp
-L Battery BT1
+L Battery-RESCUE-BSAT_-_Battery_Shield BT1
 U 1 1 574296C6
 P 10200 4650
@@
 $EndComp
 $Comp
-L Battery BT2
+L Battery-RESCUE-BSAT_-_Battery_Shield BT2
 U 1 1 5745DC06
 P 10200 5050
@@
 56 56 50 5E 5E FE 2B 80 B2 AA AA AA 5F F3 F2 F2 AA 94 B7 F8 C7 44 5E 5E 9E D2 E3 4A 89 E4 4F FC
 09 79 74 C5 E6 42 7F E2 FF 19 FE 24 92 3F D1 26 FE 24 92 3F D1 26 FE 24 92 3F D1 26 FE 0F 78 6D
-04 45 FC BA DA 0A 00 00 00 00 49 45 4E 44 AE 42 60 82 38
+04 45 FC BA DA 0A 00 00 00 00 49 45 4E 44 AE 42 60 82
 EndData
 $EndBitmap
@@
 Connection ~ 7400 3800
 Wire Wire Line
-	8150 2200 10250 2200
+	7950 2200 10250 2200
 Wire Wire Line
 	9150 1950 9100 1950
