File: pcb/sat_control_shield/kicad/BSAT - Control Shield.kicad_pcb (KiCad board)
At the start: 2 copper layers, 77 x 77 mm, 20 parts, among them P1 POWER, U1 ARDUINO_NANO_V3.0, U2 74HC4052E

Commit message: refactor(control-shield): Rediseño de la placa y corrección de error en la conmutación entre sensores de intensidad luminosa.
Parts:
- removed REF** (x8): 1pin, Connect:1pin
- ANT1: footprint Pin_Headers:Pin_Header_Angled_1x01 -> Pin_Headers:Pin_Header_Angled_1x01_Pitch2.54mm
- P1: footprint Pin_Headers:Pin_Header_Straight_1x02 -> Pin_Headers:Pin_Header_Straight_1x02_Pitch2.54mm
- moved S6 229.5 mm to (-58.5, 133.5), turned to 0 degrees
- moved S5 219.9 mm to (-59.0, 118.5), turned to 0 degrees
- moved S4 209.9 mm to (-58.0, 105.5), turned to 0 degrees
- moved S3 202.3 mm to (-59.0, 90.5), turned to 0 degrees
- moved P1 190.0 mm to (-74.5, 121.5)
- moved S7 166.9 mm to (6.00, 65.5), turned to 0 degrees
- moved U1 164.7 mm to (-19.0, 100.0), turned to 0 degrees
- moved U2 156.0 mm to (-26.5, 58.5), turned to 0 degrees
- moved S1 153.2 mm to (19.0, 112.5)
- moved S2 129.4 mm to (52.0, 106.0), turned to 0 degrees
- moved TX1 58.7 mm to (60.0, 76.5)
- moved ANT1 50.6 mm to (87.0, 67.0), turned to 0 degrees
Connections:
- S2 pad 8: Net-(S2-Pad8) -> /GYRO_INT
- U1 pad 10: /LS_SELECT_1 -> Net-(U1-Pad10)
- U1 pad 11: /LS_SELECT_0 -> Net-(U1-Pad11)
- U1 pad 20: Net-(U1-Pad20) -> /GYRO_INT
- U1 pad 21: Net-(U1-Pad21) -> /LS_SELECT_0
- U1 pad 22: Net-(U1-Pad22) -> /LS_SELECT_1
Routing:
- net GNDREF: track 298.7 -> 0.00 mm, vias 2 -> 0
- net /SCL: track 204.8 -> 0.00 mm
- net /SDA: track 142.3 -> 0.00 mm
- net +3V3: track 127.8 -> 0.00 mm
- net VCC: track 76.7 -> 0.00 mm
- net /LS_SELECT_1: track 72.6 -> 0.00 mm
- net +5V: track 66.9 -> 0.00 mm
- net /LS_SELECT_0: track 65.3 -> 0.00 mm
- net /SDA_LS_SIDE4: track 34.6 -> 0.00 mm
- net /SDA_LS_SIDE3: track 28.3 -> 0.00 mm
- net RADIO_DATA: track 26.4 -> 0.00 mm
- net /SDA_LS_SIDE2: track 25.1 -> 0.00 mm
- net (no net): track 23.1 -> 0.00 mm
- net /SDA_LS_SIDE1: track 18.6 -> 0.00 mm
- net Net-(ANT1-Pad1): track 7.05 -> 0.00 mm
- removed copper zone on B.Cu, net (none)
- removed copper zone on B.Cu, net GNDREF
Other:
- board outline removed
- board text removed: "BOSCOVERYSAT 2016 SAT CONTROL SHIELD"
- board text removed: "LIGHT SENSORS"
- board text removed: "SAT POWER"
- board text removed: "SIDE 1"
- board text removed: "SIDE 2"
- board text removed: "SIDE 3"
- board text removed: "SIDE 4"
- board text removed: "V1.1"
- board text removed: "VCC ADDR GND SCL SDA"
- board text removed: "X"
- board text removed: "Y"
